Commit message: Setup support package w URDF

File: motoman_gp180_support/urdf/gp180_120_macro.xacro (robot description, xacro)
@@ -153,4 +153,11 @@
         <child link="${prefix}base"/>
     </joint>
+  <!-- ROS-Industrial 'flange' frame.. attachment point for EEF models -->
+  <link name="${prefix}flange" />
+  <joint name="${prefix}joint_6_t-flange" type="fixed">
+    <parent link="${prefix}link_6_t" />
+    <child link="${prefix}flange" />
+    <origin xyz="0 0 0" rpy="0 0 0" />
+  </joint>
 </xacro:macro>
 </robot>
